File: hw/usb_switch/usb_switch.kicad_pcb (KiCad board)
At the start: 4 copper layers, 60 x 65 mm, 75 parts, among them J1 host_usb, J2 alt_source_usb, J3 Conn_01x02, J4 Conn_01x02, J5 Conn_01x02, J6 Conn_01x02, J7 extra_usb, J8 target_usb, U1 MIC5504-3.3YM5, U2 FSUSB30L10X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

Commit message: Finished and ordered from JLCPCB!
Parts:
- added C22: 0.1uF, Capacitor_SMD:C_0402_1005Metric, F.Cu at (82.9, 86.3)
- added REF**: OSHW-Logo2_48.7x40mm_SilkScreen, Symbol:OSHW-Logo2_48.7x40mm_SilkScreen, B.Cu at (70.5, 74.0)
- R24: value R_Small -> 1M
- R25: value R_Small -> 62k
- moved TP1 38.4 mm to (77.4, 102.5)
- moved J6 27.1 mm to (83.8, 77.2), turned to -90 degrees
- moved R12 24.1 mm to (83.3, 74.7)
- moved C17 19.2 mm to (62.9, 73.7), turned to -90 degrees
- moved R27 18.9 mm to (59.1, 98.2)
- moved J5 18.1 mm to (59.2, 72.1), turned to -90 degrees
- moved U4 18.0 mm to (65.5, 72.2), turned to 180 degrees
- moved R26 14.6 mm to (64.9, 69.9), turned to 0 degrees
- moved R29 12.3 mm to (82.9, 85.3)
- moved FB3 10.6 mm to (90.5, 57.0), turned to -90 degrees
- moved J4 9.63 mm to (83.6, 95.2), turned to 90 degrees
- moved C15 8.15 mm to (71.1, 94.1), turned to 90 degrees
- moved J3 8.10 mm to (60.5, 100.7), turned to -90 degrees
- moved R28 7.40 mm to (63.8, 80.4), turned to -90 degrees
- moved C14 7.27 mm to (71.2, 97.0), turned to -90 degrees
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Routing:
- net +5V: track 0.00 -> 110.9 mm
- net GND: track 0.00 -> 48.1 mm, vias 0 -> 47
- net /CC1: track 0.00 -> 44.9 mm, vias 0 -> 2
- net /CC2: track 0.00 -> 43.1 mm, vias 0 -> 2
- net +3V3: track 0.00 -> 40.4 mm, vias 0 -> 11
- net /USB_C_VBUS_EN_N: track 0.00 -> 35.2 mm, vias 0 -> 2
- net VBUS: track 0.00 -> 20.0 mm, vias 0 -> 8
- net Net-(FB3-Pad2): track 0.00 -> 17.7 mm
- net /usb_power/VUSB_OUT: track 0.00 -> 17.6 mm, vias 0 -> 11
- net /USB_EN_N: track 0.00 -> 13.2 mm
- net Net-(C8-Pad1): track 0.00 -> 13.1 mm
- net Net-(R22-Pad2): track 0.00 -> 11.8 mm
- net Net-(FB4-Pad2): track 0.00 -> 10.1 mm, vias 0 -> 2
- net Net-(C1-Pad1): track 0.00 -> 9.94 mm, vias 0 -> 2
- net Net-(FB2-Pad1): track 0.00 -> 9.80 mm, vias 0 -> 2
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- added copper zone on In2.Cu, net +3V3
- added copper zone on In2.Cu, net /usb_power/VUSB_OUT
- added copper zone on In1.Cu, net GND
- added copper zone on In2.Cu, net VBUS
Other:
- board size 60 x 65 mm -> 60 x 60 mm
- board text added: "Alt Power/Data"
- board text added: "DEBUGINATOR USB SWITCH"
- board text added: "Extra"
- board text added: "Host"
- board text added: "Quesadillon LLC"
- board text added: "Target"
- board text added: "USBC VBUS EN_N"
- board text added: "USB_EN"
- board text added: "USB_EN_N"
- board text added: "USB_SEL"
- board text added: "v1.0"
