File: hw/usb_switch/usb_hub.kicad_sch (KiCad schematic)
At the start: 18 parts, among them U3 TUSB2036, Y1 6MHz

Commit message: Updating footprints
Parts:
- C10, C11, C6, C7, C8: footprint (none) -> Capacitor_SMD:C_0402_1005Metric
- C9: footprint (none) -> Capacitor_SMD:C_0603_1608Metric
- R11, R12, R13, R14, R15, R16, R17, R18, R19, R20: footprint (none) -> Resistor_SMD:R_0402_1005Metric

Commit message: Some part changes and started layout
Parts:
- removed C9: 10uF, Capacitor_SMD:C_0603_1608Metric, symbol Device:C_Small
- added C11: 1uF, Capacitor_SMD:C_0402_1005Metric, symbol Device:C_Small
- Y1: footprint (none) -> Crystal:Crystal_SMD_HC49-SD
- renumbered C8 to C10, C10 to C12, C11 to C13, C6 to C8, C7 to C9, R11 to R13, R12 to R14, R13 to R15, R14 to R16, R15 to R17, R16 to R18, R17 to R19, R18 to R20, R19 to R21, R20 to R22
Connections:
- net +3V3: now also C11.1
- net GND: now also C11.2

Commit message: Added MPNs and values to usb_switch
Parts:
- U3: MPN (none) -> TUSB2036VFR
- Y1: MPN (none) -> ABLS2-6.000MHZ-D4Y-T
Changed lines of the file:
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@@
+      (effects (font (size 1.27 1.27)) hide)
+    )
+    (property "MPN" "TUSB2036VFR" (id 4) (at 144.78 96.52 0)
       (effects (font (size 1.27 1.27)) hide)
     )
@@
       (effects (font (size 1.27 1.27)) hide)
     )
+    (property "MPN" " ABLS2-6.000MHZ-D4Y-T" (id 4) (at 102.87 127 0)
+      (effects (font (size 1.27 1.27)) hide)
+    )
