File: hw/swd_over_c/swd_over_c.kicad_sch (KiCad schematic)
At the start: 22 parts, among them J1 USB_C_Receptacle_USB2.0, J2 Conn_ARM_JTAG_SWD_10, P1 USB_C_Plug, U1 ATtiny24-20M

Commit message: Updated swd over c to v1.1 (and programmer)
Parts:
- removed TP1: VBUS, alvarop:TP-1mm, symbol Connector:TestPoint
- removed TP2: GND, alvarop:TP-1mm, symbol Connector:TestPoint
- removed TP3: SCK, alvarop:TP-1mm, symbol Connector:TestPoint
- removed TP4: MISO, alvarop:TP-1mm, symbol Connector:TestPoint
- removed TP5: MOSI, alvarop:TP-1mm, symbol Connector:TestPoint
- removed TP6: NRST, alvarop:TP-1mm, symbol Connector:TestPoint
- D1: MPN (none) -> HSMG-C120
- D2: MPN (none) -> HSMC-C120
- J1: MPN (none) -> USB4105-GF-A
- J2: footprint alvarop:3220-10-0300-00 -> snapeda:SAMTEC_FTSH-105-01-F-DV-P-TR; MPN (none) -> 3220-10-0300-00
- P1: MPN (none) -> USB4155-03-C
- U1: footprint Package_DFN_QFN:QFN-20-1EP_4x4mm_P0.5mm_EP2.6x2.6mm -> ultralibrarian:ATTINY24A-MMH; MPN (none) -> ATTINY24A-MMH
Connections:
- net CC2_R1: now also U1.4 (PA1); no longer U1.14 (PB2)
- net CC2_R2: now also U1.5 (AREF/PA0); no longer U1.15 (PA7)
- net MCURST: now also J1.B8 (SBU2)
- net SBU1: now also R7.1; no longer U1.5 (AREF/PA0)
- net SBU2: now also R8.2; no longer U1.4 (PA1)
- net SCK: now also J1.A8 (SBU1)
- net CC1_IN renamed CC1_IN_MOSI
- net CC1_IN_MOSI: now also U1.16 (PA6); no longer U1.3 (PA2)
- net CC2_IN renamed CC2_IN_MISO
- net CC2_IN_MISO: now also U1.20 (PA5); no longer U1.2 (PA3)
- removed net MISO: R7.1, U1.20 (PA5)
- removed net MOSI: R8.2, U1.16 (PA6)
- no-connect marks 7 -> 9

Commit message: Switched to 0402 instead of 0201 components
Parts:
- C1, C2: footprint Capacitor_SMD:C_0201_0603Metric -> Capacitor_SMD:C_0402_1005Metric
- D1, D2: footprint alvarop:HSMx-C120 -> LED_SMD:LED_0603_1608Metric
- R1, R2, R3, R4, R5, R6, R7, R8: footprint Resistor_SMD:R_0201_0603Metric -> Resistor_SMD:R_0402_1005Metric
Changed lines of the file:
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@@
     (property "Reference" "D1" (id 0) (at 182.8165 87.63 0))
     (property "Value" "GREEN" (id 1) (at 182.8165 90.17 0))
-    (property "Footprint" "alvarop:HSMx-C120" (id 2) (at 182.88 93.98 90)
+    (property "Footprint" "LED_SMD:LED_0603_1608Metric" (id 2) (at 182.88 93.98 90)
       (effects (font (size 1.27 1.27)) hide)
     )
@@
       (effects (font (size 1.27 1.27)) (justify left))
     )
-    (property "Footprint" "Capacitor_SMD:C_0201_0603Metric" (id 2) (at 101.6 30.48 0)
+    (property "Footprint" "Capacitor_SMD:C_0402_1005Metric" (id 2) (at 101.6 30.48 0)
       (effects (font (size 1.27 1.27)) hide)
     )
@@
     (property "Reference" "R6" (id 0) (at 180.34 81.28 90))
     (property "Value" "56k" (id 1) (at 180.34 78.74 90))
-    (property "Footprint" "Resistor_SMD:R_0201_0603Metric" (id 2) (at 180.34 76.2 0)
+    (property "Footprint" "Resistor_SMD:R_0402_1005Metric" (id 2) (at 180.34 76.2 0)
       (effects (font (size 1.27 1.27)) hide)
     )
@@
     (property "Reference" "R7" (id 0) (at 175.26 88.9 90))
     (property "Value" "1k" (id 1) (at 175.26 91.44 90))
-    (property "Footprint" "Resistor_SMD:R_0201_0603Metric" (id 2) (at 175.26 93.98 0)
+    (property "Footprint" "Resistor_SMD:R_0402_1005Metric" (id 2) (at 175.26 93.98 0)
       (effects (font (size 1.27 1.27)) hide)
     )
@@
     (property "Reference" "R2" (id 0) (at 68.58 96.52 90))
     (property "Value" "5.1k" (id 1) (at 66.04 96.52 90))
-    (property "Footprint" "Resistor_SMD:R_0201_0603Metric" (id 2) (at 63.5 96.52 0)
+    (property "Footprint" "Resistor_SMD:R_0402_1005Metric" (id 2) (at 63.5 96.52 0)
       (effects (font (size 1.27 1.27)) hide)
     )
@@
     (property "Reference" "R8" (id 0) (at 175.26 104.14 90))
     (property "Value" "1k" (id 1) (at 175.26 101.6 90))
-    (property "Footprint" "Resistor_SMD:R_0201_0603Metric" (id 2) (at 175.26 99.06 0)
+    (property "Footprint" "Resistor_SMD:R_0402_1005Metric" (id 2) (at 175.26 99.06 0)
       (effects (font (size 1.27 1.27)) hide)
     )
@@
       (effects (font (size 1.27 1.27)) (justify left))
     )
-    (property "Footprint" "Capacitor_SMD:C_0201_0603Metric" (id 2) (at 91.44 30.48 0)
+    (property "Footprint" "Capacitor_SMD:C_0402_1005Metric" (id 2) (at 91.44 30.48 0)
       (effects (font (size 1.27 1.27)) hide)
     )
@@
     (property "Reference" "D2" (id 0) (at 182.88 104.14 0))
     (property "Value" "RED" (id 1) (at 182.88 101.6 0))
-    (property "Footprint" "alvarop:HSMx-C120" (id 2) (at 182.88 99.06 90)
+    (property "Footprint" "LED_SMD:LED_0603_1608Metric" (id 2) (at 182.88 99.06 90)
       (effects (font (size 1.27 1.27)) hide)
     )
@@
     (property "Reference" "R5" (id 0) (at 180.34 68.58 90))
     (property "Value" "22k" (id 1) (at 180.34 71.12 90))
-    (property "Footprint" "Resistor_SMD:R_0201_0603Metric" (id 2) (at 180.34 73.66 0)
+    (property "Footprint" "Resistor_SMD:R_0402_1005Metric" (id 2) (at 180.34 73.66 0)
       (effects (font (size 1.27 1.27)) hide)
     )
@@
     (property "Reference" "R1" (id 0) (at 55.88 96.52 90))
     (property "Value" "5.1k" (id 1) (at 58.42 96.52 90))
-    (property "Footprint" "Resistor_SMD:R_0201_0603Metric" (id 2) (at 60.96 96.52 0)
+    (property "Footprint" "Resistor_SMD:R_0402_1005Metric" (id 2) (at 60.96 96.52 0)
       (effects (font (size 1.27 1.27)) hide)
     )
@@
     (property "Reference" "R3" (id 0) (at 180.34 52.07 90))
     (property "Value" "10k" (id 1) (at 180.34 55.88 90))
-    (property "Footprint" "Resistor_SMD:R_0201_0603Metric" (id 2) (at 180.34 58.42 0)
+    (property "Footprint" "Resistor_SMD:R_0402_1005Metric" (id 2) (at 180.34 58.42 0)
       (effects (font (size 1.27 1.27)) hide)
     )
@@
     (property "Reference" "R4" (id 0) (at 180.34 66.04 90))
     (property "Value" "22k" (id 1) (at 180.34 63.5 90))
-    (property "Footprint" "Resistor_SMD:R_0201_0603Metric" (id 2) (at 180.34 60.96 0)
+    (property "Footprint" "Resistor_SMD:R_0402_1005Metric" (id 2) (at 180.34 60.96 0)
       (effects (font (size 1.27 1.27)) hide)
     )
@@
     )
     (path "/c9835c81-c2e5-419b-85f5-0bcc77b4e78f"
-      (reference "C1") (unit 1) (value "1uF") (footprint "Capacitor_SMD:C_0201_0603Metric")
+      (reference "C1") (unit 1) (value "1uF") (footprint "Capacitor_SMD:C_0402_1005Metric")
     )
     (path "/1e443a9e-89d1-4d2d-9468-44ef36b04c6b"
-      (reference "C2") (unit 1) (value "0.1uF") (footprint "Capacitor_SMD:C_0201_0603Metric")
+      (reference "C2") (unit 1) (value "0.1uF") (footprint "Capacitor_SMD:C_0402_1005Metric")
     )
     (path "/17f8dd66-03f8-44e1-8db0-4cda05e23a2b"
-      (reference "D1") (unit 1) (value "GREEN") (footprint "alvarop:HSMx-C120")
+      (reference "D1") (unit 1) (value "GREEN") (footprint "LED_SMD:LED_0603_1608Metric")
     )
     (path "/dbda3428-3d38-4a6e-871d-6f5f17b7e6e0"
-      (reference "D2") (unit 1) (value "RED") (footprint "alvarop:HSMx-C120")
+      (reference "D2") (unit 1) (value "RED") (footprint "LED_SMD:LED_0603_1608Metric")
     )
     (path "/afb8b546-2d34-49f9-b048-809d9d067ebb"
@@
     )
     (path "/de70c41d-5ffd-41c8-a48a-126c007da711"
-      (reference "R1") (unit 1) (value "5.1k") (footprint "Resistor_SMD:R_0201_0603Metric")
+      (reference "R1") (unit 1) (value "5.1k") (footprint "Resistor_SMD:R_0402_1005Metric")
     )
     (path "/8c67700b-9995-44f5-96fd-fdb8736067e6"
-      (reference "R2") (unit 1) (value "5.1k") (footprint "Resistor_SMD:R_0201_0603Metric")
+      (reference "R2") (unit 1) (value "5.1k") (footprint "Resistor_SMD:R_0402_1005Metric")
     )
     (path "/f08354d6-f42f-4f89-b816-6911e2618ed5"
-      (reference "R3") (unit 1) (value "10k") (footprint "Resistor_SMD:R_0201_0603Metric")
+      (reference "R3") (unit 1) (value "10k") (footprint "Resistor_SMD:R_0402_1005Metric")
     )
     (path "/f9423327-8224-4ffb-82f8-87802acf6581"
-      (reference "R4") (unit 1) (value "22k") (footprint "Resistor_SMD:R_0201_0603Metric")
+      (reference "R4") (unit 1) (value "22k") (footprint "Resistor_SMD:R_0402_1005Metric")
     )
     (path "/de2663d9-cfce-4455-9b8d-5ceda6e2a445"
-      (reference "R5") (unit 1) (value "22k") (footprint "Resistor_SMD:R_0201_0603Metric")
+      (reference "R5") (unit 1) (value "22k") (footprint "Resistor_SMD:R_0402_1005Metric")
     )
     (path "/4e7e97d5-569c-4054-82d8-5d403c39cdea"
-      (reference "R6") (unit 1) (value "56k") (footprint "Resistor_SMD:R_0201_0603Metric")
+      (reference "R6") (unit 1) (value "56k") (footprint "Resistor_SMD:R_0402_1005Metric")
     )
     (path "/68e7324f-c14f-43fb-b880-c73f6737944e"
-      (reference "R7") (unit 1) (value "1k") (footprint "Resistor_SMD:R_0201_0603Metric")
+      (reference "R7") (unit 1) (value "1k") (footprint "Resistor_SMD:R_0402_1005Metric")
     )
     (path "/a7c7872e-a04c-47f4-9ddf-83f77ee0e7bf"
-      (reference "R8") (unit 1) (value "1k") (footprint "Resistor_SMD:R_0201_0603Metric")
+      (reference "R8") (unit 1) (value "1k") (footprint "Resistor_SMD:R_0402_1005Metric")
     )
     (path "/c8daeb28-c525-4e55-a264-b6cb07a30f2d"

Commit message: Minor bom updates
Parts:
- D1: MPN HSMG-C120 -> (none)
- D2: MPN HSMC-C120 -> (none)
Changed lines of the file:
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@@
       (effects (font (size 1.27 1.27)) hide)
     )
-    (property "MPN" "HSMG-C120" (id 4) (at 182.88 93.98 0)
+    (property "MPN" "" (id 4) (at 182.88 93.98 0)
       (effects (font (size 1.27 1.27)) hide)
     )
@@
       (effects (font (size 1.27 1.27)) hide)
     )
-    (property "MPN" "HSMC-C120" (id 4) (at 182.88 99.06 0)
-      (effects (font (size 1.27 1.27)) hide)
-    )
+    (property "MPN" "" (id 4) (at 182.88 99.06 0)
+      (effects (font (size 1.27 1.27)) hide)
+    )

Commit message: Fixed MISO/MOSI swap and added BOM to swd2usbc
Parts:
- C1: Footprint(Generic) (none) -> C0402; MPN (none) -> CL05A105KO5NNNC; Manufacturer (none) -> Samsung Electro-Mechanics; Vendor (none) -> Digi-Key; Vendor Part Number (none) -> 1276-1067-1-ND
- C2: Footprint(Generic) (none) -> C0402; MPN (none) -> CL05B104KO5NNNC; Manufacturer (none) -> Samsung Electro-Mechanics; Vendor (none) -> Digi-Key; Vendor Part Number (none) -> 1276-1001-1-ND
- D1: Footprint(Generic) (none) -> 0603; MPN (none) -> SML-D12M8WT86; Manufacturer (none) -> Rohm Semiconductor; Vendor (none) -> Digi-Key; Vendor Part Number (none) -> 511-1578-1-ND
- D2: Footprint(Generic) (none) -> 0603; MPN (none) -> SML-D12U1WT86; Manufacturer (none) -> Rohm Semiconductor; Vendor (none) -> Digi-Key; Vendor Part Number (none) -> SML-D12U1WT86CT-ND
- J1: Footprint(Generic) (none) -> USB4105-GF-A; Manufacturer (none) -> GCT; Vendor (none) -> Digi-Key; Vendor Part Number (none) -> 2073-USB4105-GF-ACT-ND
- J2: Footprint(Generic) (none) -> SAMTEC_FTSH-105-01-F-DV-P-TR; MPN 3220-10-0300-00 -> FTSH-105-01-F-DV-K; Manufacturer (none) -> Samtec Inc.; Vendor (none) -> Digi-Key; Vendor Part Number (none) -> SAM8796-ND
- P1: footprint alvarop:‎USB4155-03-C‎ -> alvarop:MOLEX_1054440011; Footprint(Generic) (none) -> 1054440011; MPN USB4155-03-C -> 1054440011; Manufacturer (none) -> Molex; Vendor (none) -> Digi-Key; Vendor Part Number (none) -> 900-1054440011CT-ND
- R1, R2: Footprint(Generic) (none) -> R0402; MPN (none) -> RC0402FR-075K1L; Manufacturer (none) -> Yageo; Vendor (none) -> Digi-Key; Vendor Part Number (none) -> 311-5.1KJRCT-ND
- R3: Footprint(Generic) (none) -> R0402; MPN (none) -> RC0402FR-0710KL; Manufacturer (none) -> Yageo; Vendor (none) -> Digi-Key; Vendor Part Number (none) -> 311-10.0KLRCT-ND
- R4, R5: Footprint(Generic) (none) -> R0402; MPN (none) -> RC0402FR-0722KL; Manufacturer (none) -> Yageo; Vendor (none) -> Digi-Key; Vendor Part Number (none) -> 311-22.0KLRCT-ND
- R6: Footprint(Generic) (none) -> R0402; MPN (none) -> RC0402FR-0756KL; Manufacturer (none) -> Yageo; Vendor (none) -> Digi-Key; Vendor Part Number (none) -> 311-56.0KLRCT-ND
- R7, R8: Footprint(Generic) (none) -> R0402; MPN (none) -> RC0402FR-071KL; Manufacturer (none) -> Yageo; Vendor (none) -> Digi-Key; Vendor Part Number (none) -> 311-1.00KLRCT-ND
- U1: Footprint(Generic) (none) -> 20VQFN; MPN ATTINY24A-MMH -> ATTINY24A-MMH; Manufacturer (none) -> Microchip; Vendor (none) -> Digi-Key; Vendor Part Number (none) -> ATTINY24A-MMH-ND

Commit message: SWD over USB-C v1.4!!!
Parts:
- C1: value 1uF -> (none); footprint Capacitor_SMD:C_0402_1005Metric -> (none)
- C2: value 0.1uF -> (none); footprint Capacitor_SMD:C_0402_1005Metric -> (none)
- D1: value GREEN -> (none); footprint LED_SMD:LED_0603_1608Metric -> (none)
- D2: value RED -> (none); footprint LED_SMD:LED_0603_1608Metric -> (none)
- J1: value USB_C_Receptacle_USB2.0 -> (none); footprint alvarop:USB4105-GF-A -> (none); Footprint(Generic) USB4105-GF-A -> USB4500-03-0-A; MPN USB4105-GF-A -> USB4500-03-0-A; Vendor Part Number 2073-USB4105-GF-ACT-ND -> 2073-USB4500-03-0-ACT-ND
- J2: value Conn_ARM_JTAG_SWD_10 -> (none); footprint snapeda:SAMTEC_FTSH-105-01-F-DV-P-TR -> (none); Vendor Part Number SAM8796-ND -> SAM13160CT-ND
- P1: value USB_C_Plug -> (none); footprint alvarop:MOLEX_1054440011 -> (none)
- R1, R2: value 5.1k -> (none); footprint Resistor_SMD:R_0402_1005Metric -> (none)
- R3: value 10k -> (none); footprint Resistor_SMD:R_0402_1005Metric -> (none); MPN RC0402FR-0710KL -> RC0402FR-0722KL; Vendor Part Number 311-10.0KLRCT-ND -> 311-22.0KLRCT-ND
- R4: value 22k -> (none); footprint Resistor_SMD:R_0402_1005Metric -> (none); MPN RC0402FR-0722KL -> RC0402FR-0756KL; Vendor Part Number 311-22.0KLRCT-ND -> 311-56.0KLRCT-ND
- R5: value 22k -> (none); footprint Resistor_SMD:R_0402_1005Metric -> (none); MPN RC0402FR-0722KL -> RC0402FR-0710KL; Vendor Part Number 311-22.0KLRCT-ND -> 311-10.0KLRCT-ND
- R6: value 56k -> (none); footprint Resistor_SMD:R_0402_1005Metric -> (none); MPN RC0402FR-0756KL -> RC0402FR-0722KL; Vendor Part Number 311-56.0KLRCT-ND -> 311-22.0KLRCT-ND
- R7, R8: value 1k -> (none); footprint Resistor_SMD:R_0402_1005Metric -> (none)
- U1: value ATtiny24-20M -> (none); footprint ultralibrarian:ATTINY24A-MMH -> (none)
Connections:
- net CC1: now also R3.1, R4.1; no longer R3.2, R4.2
- net CC1_R1: now also R3.2; no longer R3.1
- net CC1_R2: now also R4.2; no longer R4.1
- net CC2: now also R6.2; no longer R6.1
- net CC2_R2: now also R6.1; no longer R6.2

Commit message: v1.6 changes
Parts:
- C1: value (none) -> 1uF; footprint (none) -> Capacitor_SMD:C_0402_1005Metric
- C2: value (none) -> 0.1uF; footprint (none) -> Capacitor_SMD:C_0402_1005Metric
- D1: value (none) -> GREEN; footprint (none) -> LED_SMD:LED_0603_1608Metric
- D2: value (none) -> RED; footprint (none) -> LED_SMD:LED_0603_1608Metric
- J1: value (none) -> USB_C_Receptacle_USB2.0; footprint (none) -> alvarop:USB4500-03
- J2: value (none) -> Conn_ARM_JTAG_SWD_10; footprint (none) -> snapeda:SAMTEC_FTSH-105-01-F-DV-P-TR
- P1: value (none) -> USB_C_Plug; footprint (none) -> alvarop:‎USB4155-03-C‎
- R1, R2: value (none) -> 5.1k; footprint (none) -> Resistor_SMD:R_0402_1005Metric
- R3, R6: value (none) -> 22k; footprint (none) -> Resistor_SMD:R_0402_1005Metric
- R4: value (none) -> 56k; footprint (none) -> Resistor_SMD:R_0402_1005Metric
- R5: value (none) -> 10k; footprint (none) -> Resistor_SMD:R_0402_1005Metric
- R7, R8: value (none) -> 1k; footprint (none) -> Resistor_SMD:R_0402_1005Metric
- U1: value (none) -> ATtiny24-20M; footprint (none) -> ultralibrarian:ATTINY24A-MMH_MOD
Changed lines of the file:
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@@
   (title_block
     (title "Debugotron - SWD2USBC")
-    (date "2022-03-25")
+    (date "2022-05-15")
     (rev "1.4")
     (company "Quesadillon LLC")
@@
     (in_bom yes) (on_board yes) (fields_autoplaced)
     (property "Reference" "D1" (id 0) (at 182.8165 87.63 0))
-    (property "Value" "" (id 1) (at 182.8165 90.17 0))
-    (property "Footprint" "" (id 2) (at 182.88 93.98 90)
+    (property "Value" "GREEN" (id 1) (at 182.8165 90.17 0))
+    (property "Footprint" "LED_SMD:LED_0603_1608Metric" (id 2) (at 182.88 93.98 90)
       (effects (font (size 1.27 1.27)) hide)
     )
@@
       (effects (font (size 1.27 1.27)) (justify left))
     )
-    (property "Value" "" (id 1) (at 104.14 31.7562 0)
+    (property "Value" "0.1uF" (id 1) (at 104.14 31.7562 0)
       (effects (font (size 1.27 1.27)) (justify left))
     )
-    (property "Footprint" "" (id 2) (at 101.6 30.48 0)
+    (property "Footprint" "Capacitor_SMD:C_0402_1005Metric" (id 2) (at 101.6 30.48 0)
       (effects (font (size 1.27 1.27)) hide)
     )
@@
     (in_bom yes) (on_board yes)
     (property "Reference" "R6" (id 0) (at 180.34 81.28 90))
-    (property "Value" "" (id 1) (at 180.34 78.74 90))
-    (property "Footprint" "" (id 2) (at 180.34 76.2 0)
+    (property "Value" "22k" (id 1) (at 180.34 78.74 90))
+    (property "Footprint" "Resistor_SMD:R_0402_1005Metric" (id 2) (at 180.34 76.2 0)
       (effects (font (size 1.27 1.27)) hide)
     )
@@
     (in_bom yes) (on_board yes)
     (property "Reference" "R5" (id 0) (at 180.34 67.31 90))
-    (property "Value" "" (id 1) (at 180.34 71.12 90))
-    (property "Footprint" "" (id 2) (at 180.34 73.66 0)
+    (property "Value" "10k" (id 1) (at 180.34 71.12 90))
+    (property "Footprint" "Resistor_SMD:R_0402_1005Metric" (id 2) (at 180.34 73.66 0)
       (effects (font (size 1.27 1.27)) hide)
     )
@@
     (in_bom yes) (on_board yes)
     (property "Reference" "R4" (id 0) (at 180.34 66.04 90))
-    (property "Value" "" (id 1) (at 180.34 63.5 90))
-    (property "Footprint" "" (id 2) (at 180.34 60.96 0)
+    (property "Value" "56k" (id 1) (at 180.34 63.5 90))
+    (property "Footprint" "Resistor_SMD:R_0402_1005Metric" (id 2) (at 180.34 60.96 0)
       (effects (font (size 1.27 1.27)) hide)
     )
@@
     (in_bom yes) (on_board yes)
     (property "Reference" "R7" (id 0) (at 175.26 88.9 90))
-    (property "Value" "" (id 1) (at 175.26 91.44 90))
-    (property "Footprint" "" (id 2) (at 175.26 93.98 0)
+    (property "Value" "1k" (id 1) (at 175.26 91.44 90))
+    (property "Footprint" "Resistor_SMD:R_0402_1005Metric" (id 2) (at 175.26 93.98 0)
       (effects (font (size 1.27 1.27)) hide)
     )
@@
       (effects (font (size 1.27 1.27)) (justify right))
     )
-    (property "Value" "" (id 1) (at 270.51 93.9799 0)
+    (property "Value" "USB_C_Plug" (id 1) (at 270.51 93.9799 0)
       (effects (font (size 1.27 1.27)) (justify right))
     )
-    (property "Footprint" "" (id 2) (at 255.27 88.9 0)
+    (property "Footprint" "alvarop:‎USB4155-03-C‎" (id 2) (at 255.27 88.9 0)
       (effects (font (size 1.27 1.27)) hide)
     )
@@
     (in_bom yes) (on_board yes)
     (property "Reference" "R3" (id 0) (at 180.34 53.34 90))
-    (property "Value" "" (id 1) (at 180.34 55.88 90))
-    (property "Footprint" "" (id 2) (at 180.34 58.42 0)
+    (property "Value" "22k" (id 1) (at 180.34 55.88 90))
+    (property "Footprint" "Resistor_SMD:R_0402_1005Metric" (id 2) (at 180.34 58.42 0)
       (effects (font (size 1.27 1.27)) hide)
     )
@@
     (in_bom yes) (on_board yes)
     (property "Reference" "R2" (id 0) (at 68.58 96.52 90))
-    (property "Value" "" (id 1) (at 66.04 96.52 90))
-    (property "Footprint" "" (id 2) (at 63.5 96.52 0)
+    (property "Value" "5.1k" (id 1) (at 66.04 96.52 90))
+    (property "Footprint" "Resistor_SMD:R_0402_1005Metric" (id 2) (at 63.5 96.52 0)
       (effects (font (size 1.27 1.27)) hide)
     )
@@
     (in_bom yes) (on_board yes)
     (property "Reference" "R8" (id 0) (at 175.26 104.14 90))
-    (property "Value" "" (id 1) (at 175.26 101.6 90))
-    (property "Footprint" "" (id 2) (at 175.26 99.06 0)
+    (property "Value" "1k" (id 1) (at 175.26 101.6 90))
+    (property "Footprint" "Resistor_SMD:R_0402_1005Metric" (id 2) (at 175.26 99.06 0)
       (effects (font (size 1.27 1.27)) hide)
     )
@@
       (effects (font (size 1.27 1.27)) (justify right))
     )
-    (property "Value" "" (id 1) (at 110.49 161.2899 0)
+    (property "Value" "Conn_ARM_JTAG_SWD_10" (id 1) (at 110.49 161.2899 0)
       (effects (font (size 1.27 1.27)) (justify right))
     )
-    (property "Footprint" "" (id 2) (at 121.92 160.02 0)
+    (property "Footprint" "snapeda:SAMTEC_FTSH-105-01-F-DV-P-TR" (id 2) (at 121.92 160.02 0)
       (effects (font (size 1.27 1.27)) hide)
     )
@@
     (in_bom yes) (on_board yes) (fields_autoplaced)
     (property "Reference" "J1" (id 0) (at 30.48 73.66 0))
-    (property "Value" "" (id 1) (at 30.48 76.2 0))
-    (property "Footprint" "" (id 2) (at 34.29 96.52 0)
+    (property "Value" "USB_C_Receptacle_USB2.0" (id 1) (at 30.48 76.2 0))
+    (property "Footprint" "alvarop:USB4500-03" (id 2) (at 34.29 96.52 0)
       (effects (font (size 1.27 1.27)) hide)
     )
@@
       (effects (font (size 1.27 1.27)) (justify right))
     )
-    (property "Value" "" (id 1) (at 107.95 59.6899 0)
+    (property "Value" "ATtiny24-20M" (id 1) (at 107.95 59.6899 0)
       (effects (font (size 1.27 1.27)) (justify right))
     )
-    (property "Footprint" "" (id 2) (at 121.92 58.42 0)
+    (property "Footprint" "ultralibrarian:ATTINY24A-MMH_MOD" (id 2) (at 121.92 58.42 0)
       (effects (font (size 1.27 1.27) italic) hide)
     )
@@
       (effects (font (size 1.27 1.27)) (justify left))
     )
-    (property "Value" "" (id 1) (at 93.98 31.7562 0)
+    (property "Value" "1uF" (id 1) (at 93.98 31.7562 0)
       (effects (font (size 1.27 1.27)) (justify left))
     )
-    (property "Footprint" "" (id 2) (at 91.44 30.48 0)
+    (property "Footprint" "Capacitor_SMD:C_0402_1005Metric" (id 2) (at 91.44 30.48 0)
       (effects (font (size 1.27 1.27)) hide)
     )
@@
     (in_bom yes) (on_board yes)
     (property "Reference" "D2" (id 0) (at 182.88 104.14 0))
-    (property "Value" "" (id 1) (at 182.88 101.6 0))
-    (property "Footprint" "" (id 2) (at 182.88 99.06 90)
+    (property "Value" "RED" (id 1) (at 182.88 101.6 0))
+    (property "Footprint" "LED_SMD:LED_0603_1608Metric" (id 2) (at 182.88 99.06 90)
       (effects (font (size 1.27 1.27)) hide)
     )
@@
     (in_bom yes) (on_board yes)
     (property "Reference" "R1" (id 0) (at 55.88 96.52 90))
-    (property "Value" "" (id 1) (at 58.42 96.52 90))
-    (property "Footprint" "" (id 2) (at 60.96 96.52 0)
+    (property "Value" "5.1k" (id 1) (at 58.42 96.52 90))
+    (property "Footprint" "Resistor_SMD:R_0402_1005Metric" (id 2) (at 60.96 96.52 0)
       (effects (font (size 1.27 1.27)) hide)
     )
@@
     )
     (path "/7d2422a2-6679-4b2f-b253-47eef0da2414"
-      (reference "P1") (unit 1) (value "USB_C_Plug") (footprint "alvarop:MOLEX_1054440011")
+      (reference "P1") (unit 1) (value "USB_C_Plug") (footprint "alvarop:‎USB4155-03-C‎")
     )
     (path "/de70c41d-5ffd-41c8-a48a-126c007da711"
