File: hw/swd_over_c/swd_over_c.kicad_sch (KiCad schematic)
At the start: 16 parts, among them J1 USB_C_Receptacle_USB2.0, J2 Conn_ARM_JTAG_SWD_10, P1 USB_C_Plug, U1 ATtiny24-20M

Commit message: forgot the schematic changes
Parts:
- P1: Footprint(Generic) 1054440011 -> USB4155-03-C; MPN 1054440011 -> USB4155-03-C; Manufacturer Molex -> GCT; Vendor Part Number 900-1054440011CT-ND -> 2073-USB4155-03-CCT-ND
Changed lines of the file:
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@@
       (effects (font (size 1.27 1.27)) hide)
     )
-    (property "MPN" "1054440011" (id 4) (at 259.08 88.9 0)
+    (property "MPN" "USB4155-03-C" (id 4) (at 259.08 88.9 0)
       (effects (font (size 1.27 1.27)) hide)
     )
-    (property "Description" "CONN PLUG USB3.1 TYPEC BRD EDGE" (id 5) (at 259.08 88.9 0)
+    (property "Description" "USB TYPE C, PLUG, SMT , G/F, RIG" (id 5) (at 259.08 88.9 0)
       (effects (font (size 1.27 1.27)) hide)
     )
-    (property "Footprint(Generic)" "1054440011" (id 6) (at 259.08 88.9 0)
+    (property "Footprint(Generic)" "USB4155-03-C" (id 6) (at 259.08 88.9 0)
       (effects (font (size 1.27 1.27)) hide)
     )
-    (property "Manufacturer" "Molex" (id 7) (at 259.08 88.9 0)
+    (property "Manufacturer" "GCT" (id 7) (at 259.08 88.9 0)
       (effects (font (size 1.27 1.27)) hide)
     )
@@
       (effects (font (size 1.27 1.27)) hide)
     )
-    (property "Vendor Part Number" "900-1054440011CT-ND" (id 9) (at 259.08 88.9 0)
+    (property "Vendor Part Number" "2073-USB4155-03-CCT-ND" (id 9) (at 259.08 88.9 0)
       (effects (font (size 1.27 1.27)) hide)
     )
